Commit message: UPDATE: asset file

File: source/pianist/data/robots/shadow_hand/urdf/shadow_hand_left_translation.urdf (robot description, URDF)
Before this commit: robot shadow_right, 33 links, 32 joints
Links:
- added link forearm_x_translation
- added link forearm_y_translation
- link ffdistal: geometry collision mesh filename=meshes/collision/f_distal_pst.obj scale=0.001 0.001 0.001; visual mesh filename=meshes/visual/f_distal_pst.obj scale=0.001 0.001 0.001
- link ffknuckle: geometry collision mesh filename=meshes/collision/f_knuckle_E3M5.obj; visual mesh filename=meshes/visual/f_knuckle_E3M5.obj scale=0.001 0.001 0.001
- link ffmiddle: geometry collision cylinder length=0.025 radius=0.007; collision sphere radius=0.007
- link ffproximal: geometry collision cylinder length=0.040 radius=0.007; visual mesh filename=meshes/visual/f_proximal_E3M5.obj scale=0.001 0.001 0.001
- link forearm: geometry collision box size=0.07 0.07 0.07; collision mesh filename=meshes/collision/forearm_E3M5.obj scale=0.001 0.001 0.001
- link lfdistal: geometry collision mesh filename=meshes/visual/f_distal_pst.obj scale=0.001 0.001 0.001; visual mesh filename=meshes/visual/f_distal_pst.obj scale=0.001 0.001 0.001
- link lfknuckle: geometry collision mesh filename=meshes/collision/f_knuckle_E3M5.obj; visual mesh filename=meshes/visual/f_knuckle_E3M5.obj scale=0.001 0.001 0.001
- link lfmetacarpal: geometry collision box size=0.018 0.024 0.040; visual mesh filename=meshes/visual/lf_metacarpal_E3M5_left.obj scale=0.001 0.001 0.001
- link lfmiddle: geometry collision cylinder length=0.025 radius=0.007; collision sphere radius=0.007
- link lfproximal: geometry collision cylinder length=0.040 radius=0.007; visual mesh filename=meshes/visual/f_proximal_E3M5.obj scale=0.001 0.001 0.001
- link mfdistal: geometry collision mesh filename=meshes/collision/f_distal_pst.obj scale=0.001 0.001 0.001; visual mesh filename=meshes/visual/f_distal_pst.obj scale=0.001 0.001 0.001
- link mfknuckle: geometry collision mesh filename=meshes/collision/f_knuckle_E3M5.obj; visual mesh filename=meshes/visual/f_knuckle_E3M5.obj scale=0.001 0.001 0.001
- link mfmiddle: geometry collision cylinder length=0.025 radius=0.007; collision sphere radius=0.007
- link mfproximal: geometry collision cylinder length=0.040 radius=0.007; visual mesh filename=meshes/visual/f_proximal_E3M5.obj scale=0.001 0.001 0.001
- link palm: geometry collision box size=0.018 0.024 0.004; collision box size=0.020 0.024 0.032
- link rfdistal: geometry collision mesh filename=meshes/collision/f_distal_pst.obj scale=0.001 0.001 0.001; visual mesh filename=meshes/visual/f_distal_pst.obj scale=0.001 0.001 0.001
- link rfknuckle: geometry collision mesh filename=meshes/collision/f_knuckle_E3M5.obj; visual mesh filename=meshes/visual/f_knuckle_E3M5.obj scale=0.001 0.001 0.001
- link rfmiddle: geometry collision cylinder length=0.025 radius=0.007; collision sphere radius=0.007
- link rfproximal: geometry collision cylinder length=0.040 radius=0.007; visual mesh filename=meshes/visual/f_proximal_E3M5.obj scale=0.001 0.001 0.001
- link thdistal: geometry collision mesh filename=meshes/visual/th_distal_pst.obj scale=0.001 0.001 0.001; visual mesh filename=meshes/visual/th_distal_pst.obj scale=0.001 0.001 0.001
- link thmiddle: geometry collision mesh filename=meshes/collision/th_middle_E3M5.obj scale=0.001 0.001 0.001; visual mesh filename=meshes/visual/th_middle_E3M5.obj scale=0.001 0.001 0.001
- link thproximal: geometry collision mesh filename=meshes/collision/th_proximal_E3M5.obj scale=0.001 0.001 0.001; visual mesh filename=meshes/visual/th_proximal_E3M5.obj scale=0.001 0.001 0.001
- link wrist: geometry collision box size=0.027 0.018 0.010; collision box size=0.027 0.018 0.010
Joints:
- added joint WRJX: type prismatic, parent forearm_x_translation, child forearm_y_translation, origin xyz=0.0 0.0 0.0 rpy=0.0 0.0 0.0, axis 0 0 1, limit lower=-0.5 upper=0.5 effort=10 velocity=5
- added joint WRJY: type prismatic, parent forearm_y_translation, child forearm, origin xyz=0.0 0.0 0.0 rpy=0.0 0.0 0.0, axis 1 0 0, limit lower=-0.5 upper=0.5 effort=10 velocity=5
- joint FFJ4: axis 0 -1 0 -> 0 1 0; origin xyz=0.033 0 0.095 rpy=0 0 0 -> xyz=-0.033 0 0.095 rpy=0 0 0
- joint LFJ4: axis 0 1 0 -> 0 -1 0; origin xyz=0.05397275 0 0.03779463 rpy=0 0.9599 0 -> xyz=-0.05397275 0 0.03779463 rpy=0 -0.9599 0
- joint LFJ5: origin xyz=-0.033 0 0.02071 rpy=0 -0.9599 0 -> xyz=0.033 0 0.02071 rpy=0 0.9599 0
- joint MFJ4: axis 0 -1 0 -> 0 1 0; origin xyz=0.011 0 0.099 rpy=0 0 0 -> xyz=-0.011 0 0.099 rpy=0 0 0
- joint RFJ4: axis 0 1 0 -> 0 -1 0; origin xyz=-0.011 0 0.095 rpy=0 0 0 -> xyz=0.011 0 0.095 rpy=0 0 0
- joint THJ3: axis 0 1 0 -> 0 -1 0
- joint THJ4: axis 0 1 0 -> 0 -1 0
- joint THJ5: axis 0 0 -1 -> 0 0 1; origin xyz=0.034 -0.00858 0.029 rpy=-0.785398163397 0 -1.57079632679 -> xyz=-0.034 -0.00858 0.029 rpy=-0.785398163397 0 1.57079632679
- joint WRJ2: axis 0 1 0 -> 0 -1 0
- joint ee_fixed_joint: origin xyz=0.0 0.0 0.0 rpy=0.0 0.0 -1.57079 -> xyz=0.0 0.0 0.00 rpy=0.0 0.0 0.0
- joint world_joint: child forearm -> forearm_x_translation; origin xyz=0.0 0.0 0.0 rpy=0.0 0.0 1.57079 -> xyz=0.0 0.0 0.0 rpy=1.57079 0.0 1.57079
