Commit message: FIX: piano asset

File: source/pianist/data/assets/piano/urdf/piano.urdf (robot description, URDF)
Before this commit: robot piano, 89 links, 88 joints
Links:
- added link body, mass 10.0; collision box size=0.1 1.2209999999999999 0.04; visual box size=0.1 1.2209999999999999 0.04
- link base: mass 10.0 -> None; geometry 
- link black_key_1: geometry collision box size=0.09 0.01 0.018; visual box size=0.09 0.01 0.018
- link black_key_11: geometry collision box size=0.09 0.01 0.018; visual box size=0.09 0.01 0.018
- link black_key_13: geometry collision box size=0.09 0.01 0.018; visual box size=0.09 0.01 0.018
- link black_key_16: geometry collision box size=0.09 0.01 0.018; visual box size=0.09 0.01 0.018
- link black_key_18: geometry collision box size=0.09 0.01 0.018; visual box size=0.09 0.01 0.018
- link black_key_21: geometry collision box size=0.09 0.01 0.018; visual box size=0.09 0.01 0.018
- link black_key_23: geometry collision box size=0.09 0.01 0.018; visual box size=0.09 0.01 0.018
- link black_key_25: geometry collision box size=0.09 0.01 0.018; visual box size=0.09 0.01 0.018
- link black_key_28: geometry collision box size=0.09 0.01 0.018; visual box size=0.09 0.01 0.018
- link black_key_30: geometry collision box size=0.09 0.01 0.018; visual box size=0.09 0.01 0.018
- link black_key_33: geometry collision box size=0.09 0.01 0.018; visual box size=0.09 0.01 0.018
- link black_key_35: geometry collision box size=0.09 0.01 0.018; visual box size=0.09 0.01 0.018
- link black_key_37: geometry collision box size=0.09 0.01 0.018; visual box size=0.09 0.01 0.018
- link black_key_4: geometry collision box size=0.09 0.01 0.018; visual box size=0.09 0.01 0.018
- link black_key_40: geometry collision box size=0.09 0.01 0.018; visual box size=0.09 0.01 0.018
- link black_key_42: geometry collision box size=0.09 0.01 0.018; visual box size=0.09 0.01 0.018
- link black_key_45: geometry collision box size=0.09 0.01 0.018; visual box size=0.09 0.01 0.018
- link black_key_47: geometry collision box size=0.09 0.01 0.018; visual box size=0.09 0.01 0.018
- link black_key_49: geometry collision box size=0.09 0.01 0.018; visual box size=0.09 0.01 0.018
- link black_key_52: geometry collision box size=0.09 0.01 0.018; visual box size=0.09 0.01 0.018
- link black_key_54: geometry collision box size=0.09 0.01 0.018; visual box size=0.09 0.01 0.018
- link black_key_57: geometry collision box size=0.09 0.01 0.018; visual box size=0.09 0.01 0.018
- link black_key_59: geometry collision box size=0.09 0.01 0.018; visual box size=0.09 0.01 0.018
- link black_key_6: geometry collision box size=0.09 0.01 0.018; visual box size=0.09 0.01 0.018
- link black_key_61: geometry collision box size=0.09 0.01 0.018; visual box size=0.09 0.01 0.018
- link black_key_64: geometry collision box size=0.09 0.01 0.018; visual box size=0.09 0.01 0.018
- link black_key_66: geometry collision box size=0.09 0.01 0.018; visual box size=0.09 0.01 0.018
- link black_key_69: geometry collision box size=0.09 0.01 0.018; visual box size=0.09 0.01 0.018
- link black_key_71: geometry collision box size=0.09 0.01 0.018; visual box size=0.09 0.01 0.018
- link black_key_73: geometry collision box size=0.09 0.01 0.018; visual box size=0.09 0.01 0.018
- link black_key_76: geometry collision box size=0.09 0.01 0.018; visual box size=0.09 0.01 0.018
- link black_key_78: geometry collision box size=0.09 0.01 0.018; visual box size=0.09 0.01 0.018
- link black_key_81: geometry collision box size=0.09 0.01 0.018; visual box size=0.09 0.01 0.018
- link black_key_83: geometry collision box size=0.09 0.01 0.018; visual box size=0.09 0.01 0.018
- link black_key_85: geometry collision box size=0.09 0.01 0.018; visual box size=0.09 0.01 0.018
- link black_key_9: geometry collision box size=0.09 0.01 0.018; visual box size=0.09 0.01 0.018
- link white_key_0: mass 0.040000000000000001 -> 0.04; geometry collision box size=0.15 0.0225 0.0225; visual box size=0.15 0.0225 0.0225
- link white_key_10: mass 0.040000000000000001 -> 0.04; geometry collision box size=0.15 0.0225 0.0225; visual box size=0.15 0.0225 0.0225
- link white_key_12: mass 0.040000000000000001 -> 0.04; geometry collision box size=0.15 0.0225 0.0225; visual box size=0.15 0.0225 0.0225
- link white_key_14: mass 0.040000000000000001 -> 0.04; geometry collision box size=0.15 0.0225 0.0225; visual box size=0.15 0.0225 0.0225
- link white_key_15: mass 0.040000000000000001 -> 0.04; geometry collision box size=0.15 0.0225 0.0225; visual box size=0.15 0.0225 0.0225
- link white_key_17: mass 0.040000000000000001 -> 0.04; geometry collision box size=0.15 0.0225 0.0225; visual box size=0.15 0.0225 0.0225
- link white_key_19: mass 0.040000000000000001 -> 0.04; geometry collision box size=0.15 0.0225 0.0225; visual box size=0.15 0.0225 0.0225
- link white_key_2: mass 0.040000000000000001 -> 0.04; geometry collision box size=0.15 0.0225 0.0225; visual box size=0.15 0.0225 0.0225
- link white_key_20: mass 0.040000000000000001 -> 0.04; geometry collision box size=0.15 0.0225 0.0225; visual box size=0.15 0.0225 0.0225
- link white_key_22: mass 0.040000000000000001 -> 0.04; geometry collision box size=0.15 0.0225 0.0225; visual box size=0.15 0.0225 0.0225
- link white_key_24: mass 0.040000000000000001 -> 0.04; geometry collision box size=0.15 0.0225 0.0225; visual box size=0.15 0.0225 0.0225
- link white_key_26: mass 0.040000000000000001 -> 0.04; geometry collision box size=0.15 0.0225 0.0225; visual box size=0.15 0.0225 0.0225
- link white_key_27: mass 0.040000000000000001 -> 0.04; geometry collision box size=0.15 0.0225 0.0225; visual box size=0.15 0.0225 0.0225
- link white_key_29: mass 0.040000000000000001 -> 0.04; geometry collision box size=0.15 0.0225 0.0225; visual box size=0.15 0.0225 0.0225
- link white_key_3: mass 0.040000000000000001 -> 0.04; geometry collision box size=0.15 0.0225 0.0225; visual box size=0.15 0.0225 0.0225
- link white_key_31: mass 0.040000000000000001 -> 0.04; geometry collision box size=0.15 0.0225 0.0225; visual box size=0.15 0.0225 0.0225
- link white_key_32: mass 0.040000000000000001 -> 0.04; geometry collision box size=0.15 0.0225 0.0225; visual box size=0.15 0.0225 0.0225
- link white_key_34: mass 0.040000000000000001 -> 0.04; geometry collision box size=0.15 0.0225 0.0225; visual box size=0.15 0.0225 0.0225
- link white_key_36: mass 0.040000000000000001 -> 0.04; geometry collision box size=0.15 0.0225 0.0225; visual box size=0.15 0.0225 0.0225
- link white_key_38: mass 0.040000000000000001 -> 0.04; geometry collision box size=0.15 0.0225 0.0225; visual box size=0.15 0.0225 0.0225
- link white_key_39: mass 0.040000000000000001 -> 0.04; geometry collision box size=0.15 0.0225 0.0225; visual box size=0.15 0.0225 0.0225
- link white_key_41: mass 0.040000000000000001 -> 0.04; geometry collision box size=0.15 0.0225 0.0225; visual box size=0.15 0.0225 0.0225
- link white_key_43: mass 0.040000000000000001 -> 0.04; geometry collision box size=0.15 0.0225 0.0225; visual box size=0.15 0.0225 0.0225
- link white_key_44: mass 0.040000000000000001 -> 0.04; geometry collision box size=0.15 0.0225 0.0225; visual box size=0.15 0.0225 0.0225
- link white_key_46: mass 0.040000000000000001 -> 0.04; geometry collision box size=0.15 0.0225 0.0225; visual box size=0.15 0.0225 0.0225
- link white_key_48: mass 0.040000000000000001 -> 0.04; geometry collision box size=0.15 0.0225 0.0225; visual box size=0.15 0.0225 0.0225
- link white_key_5: mass 0.040000000000000001 -> 0.04; geometry collision box size=0.15 0.0225 0.0225; visual box size=0.15 0.0225 0.0225
- link white_key_50: mass 0.040000000000000001 -> 0.04; geometry collision box size=0.15 0.0225 0.0225; visual box size=0.15 0.0225 0.0225
- link white_key_51: mass 0.040000000000000001 -> 0.04; geometry collision box size=0.15 0.0225 0.0225; visual box size=0.15 0.0225 0.0225
- link white_key_53: mass 0.040000000000000001 -> 0.04; geometry collision box size=0.15 0.0225 0.0225; visual box size=0.15 0.0225 0.0225
- link white_key_55: mass 0.040000000000000001 -> 0.04; geometry collision box size=0.15 0.0225 0.0225; visual box size=0.15 0.0225 0.0225
- link white_key_56: mass 0.040000000000000001 -> 0.04; geometry collision box size=0.15 0.0225 0.0225; visual box size=0.15 0.0225 0.0225
- link white_key_58: mass 0.040000000000000001 -> 0.04; geometry collision box size=0.15 0.0225 0.0225; visual box size=0.15 0.0225 0.0225
- link white_key_60: mass 0.040000000000000001 -> 0.04; geometry collision box size=0.15 0.0225 0.0225; visual box size=0.15 0.0225 0.0225
- link white_key_62: mass 0.040000000000000001 -> 0.04; geometry collision box size=0.15 0.0225 0.0225; visual box size=0.15 0.0225 0.0225
- link white_key_63: mass 0.040000000000000001 -> 0.04; geometry collision box size=0.15 0.0225 0.0225; visual box size=0.15 0.0225 0.0225
- link white_key_65: mass 0.040000000000000001 -> 0.04; geometry collision box size=0.15 0.0225 0.0225; visual box size=0.15 0.0225 0.0225
- link white_key_67: mass 0.040000000000000001 -> 0.04; geometry collision box size=0.15 0.0225 0.0225; visual box size=0.15 0.0225 0.0225
- link white_key_68: mass 0.040000000000000001 -> 0.04; geometry collision box size=0.15 0.0225 0.0225; visual box size=0.15 0.0225 0.0225
- link white_key_7: mass 0.040000000000000001 -> 0.04; geometry collision box size=0.15 0.0225 0.0225; visual box size=0.15 0.0225 0.0225
- link white_key_70: mass 0.040000000000000001 -> 0.04; geometry collision box size=0.15 0.0225 0.0225; visual box size=0.15 0.0225 0.0225
- link white_key_72: mass 0.040000000000000001 -> 0.04; geometry collision box size=0.15 0.0225 0.0225; visual box size=0.15 0.0225 0.0225
- link white_key_74: mass 0.040000000000000001 -> 0.04; geometry collision box size=0.15 0.0225 0.0225; visual box size=0.15 0.0225 0.0225
- link white_key_75: mass 0.040000000000000001 -> 0.04; geometry collision box size=0.15 0.0225 0.0225; visual box size=0.15 0.0225 0.0225
- link white_key_77: mass 0.040000000000000001 -> 0.04; geometry collision box size=0.15 0.0225 0.0225; visual box size=0.15 0.0225 0.0225
- link white_key_79: mass 0.040000000000000001 -> 0.04; geometry collision box size=0.15 0.0225 0.0225; visual box size=0.15 0.0225 0.0225
- link white_key_8: mass 0.040000000000000001 -> 0.04; geometry collision box size=0.15 0.0225 0.0225; visual box size=0.15 0.0225 0.0225
- link white_key_80: mass 0.040000000000000001 -> 0.04; geometry collision box size=0.15 0.0225 0.0225; visual box size=0.15 0.0225 0.0225
- link white_key_82: mass 0.040000000000000001 -> 0.04; geometry collision box size=0.15 0.0225 0.0225; visual box size=0.15 0.0225 0.0225
- link white_key_84: mass 0.040000000000000001 -> 0.04; geometry collision box size=0.15 0.0225 0.0225; visual box size=0.15 0.0225 0.0225
- link white_key_86: mass 0.040000000000000001 -> 0.04; geometry collision box size=0.15 0.0225 0.0225; visual box size=0.15 0.0225 0.0225
- link white_key_87: mass 0.040000000000000001 -> 0.04; geometry collision box size=0.15 0.0225 0.0225; visual box size=0.15 0.0225 0.0225
Joints:
- added joint base_body_joint: type fixed, parent base, child body, origin xyz=0 0 0 rpy=0 0 0
- joint black_key_11_joint: limit lower=0 upper=0.088655881867437475 effort=10.00 velocity=6.67 -> lower=0 upper=0.08865588186743747 effort=10.00 velocity=6.67; origin xyz=-0.03 -0.4459999999999999 0.026000000000000002 rpy=0 0 0 -> xyz=-0.075 -0.4459999999999999 0.026000000000000002 rpy=0 0 0
- joint black_key_13_joint: limit lower=0 upper=0.088655881867437475 effort=10.00 velocity=6.67 -> lower=0 upper=0.08865588186743747 effort=10.00 velocity=6.67; origin xyz=-0.03 -0.42249999999999993 0.026000000000000002 rpy=0 0 0 -> xyz=-0.075 -0.42249999999999993 0.026000000000000002 rpy=0 0 0
- joint black_key_16_joint: limit lower=0 upper=0.088655881867437475 effort=10.00 velocity=6.67 -> lower=0 upper=0.08865588186743747 effort=10.00 velocity=6.67; origin xyz=-0.03 -0.37549999999999994 0.026000000000000002 rpy=0 0 0 -> xyz=-0.075 -0.37549999999999994 0.026000000000000002 rpy=0 0 0
- joint black_key_18_joint: limit lower=0 upper=0.088655881867437475 effort=10.00 velocity=6.67 -> lower=0 upper=0.08865588186743747 effort=10.00 velocity=6.67; origin xyz=-0.03 -0.35199999999999987 0.026000000000000002 rpy=0 0 0 -> xyz=-0.075 -0.35199999999999987 0.026000000000000002 rpy=0 0 0
- joint black_key_1_joint: limit lower=0 upper=0.088655881867437475 effort=10.00 velocity=6.67 -> lower=0 upper=0.08865588186743747 effort=10.00 velocity=6.67; origin xyz=-0.03 -0.5875 0.026000000000000002 rpy=0 0 0 -> xyz=-0.075 -0.5875 0.026000000000000002 rpy=0 0 0
- joint black_key_21_joint: limit lower=0 upper=0.088655881867437475 effort=10.00 velocity=6.67 -> lower=0 upper=0.08865588186743747 effort=10.00 velocity=6.67; origin xyz=-0.03 -0.30499999999999994 0.026000000000000002 rpy=0 0 0 -> xyz=-0.075 -0.30499999999999994 0.026000000000000002 rpy=0 0 0
- joint black_key_23_joint: limit lower=0 upper=0.088655881867437475 effort=10.00 velocity=6.67 -> lower=0 upper=0.08865588186743747 effort=10.00 velocity=6.67; origin xyz=-0.03 -0.28149999999999986 0.026000000000000002 rpy=0 0 0 -> xyz=-0.075 -0.28149999999999986 0.026000000000000002 rpy=0 0 0
- joint black_key_25_joint: limit lower=0 upper=0.088655881867437475 effort=10.00 velocity=6.67 -> lower=0 upper=0.08865588186743747 effort=10.00 velocity=6.67; origin xyz=-0.03 -0.2579999999999999 0.026000000000000002 rpy=0 0 0 -> xyz=-0.075 -0.2579999999999999 0.026000000000000002 rpy=0 0 0
- joint black_key_28_joint: limit lower=0 upper=0.088655881867437475 effort=10.00 velocity=6.67 -> lower=0 upper=0.08865588186743747 effort=10.00 velocity=6.67; origin xyz=-0.03 -0.21099999999999997 0.026000000000000002 rpy=0 0 0 -> xyz=-0.075 -0.21099999999999997 0.026000000000000002 rpy=0 0 0
- joint black_key_30_joint: limit lower=0 upper=0.088655881867437475 effort=10.00 velocity=6.67 -> lower=0 upper=0.08865588186743747 effort=10.00 velocity=6.67; origin xyz=-0.03 -0.1874999999999999 0.026000000000000002 rpy=0 0 0 -> xyz=-0.075 -0.1874999999999999 0.026000000000000002 rpy=0 0 0
- joint black_key_33_joint: limit lower=0 upper=0.088655881867437475 effort=10.00 velocity=6.67 -> lower=0 upper=0.08865588186743747 effort=10.00 velocity=6.67; origin xyz=-0.03 -0.14049999999999996 0.026000000000000002 rpy=0 0 0 -> xyz=-0.075 -0.14049999999999996 0.026000000000000002 rpy=0 0 0
- joint black_key_35_joint: limit lower=0 upper=0.088655881867437475 effort=10.00 velocity=6.67 -> lower=0 upper=0.08865588186743747 effort=10.00 velocity=6.67; origin xyz=-0.03 -0.11699999999999988 0.026000000000000002 rpy=0 0 0 -> xyz=-0.075 -0.11699999999999988 0.026000000000000002 rpy=0 0 0
- joint black_key_37_joint: limit lower=0 upper=0.088655881867437475 effort=10.00 velocity=6.67 -> lower=0 upper=0.08865588186743747 effort=10.00 velocity=6.67; origin xyz=-0.03 -0.09349999999999992 0.026000000000000002 rpy=0 0 0 -> xyz=-0.075 -0.09349999999999992 0.026000000000000002 rpy=0 0 0
- joint black_key_40_joint: limit lower=0 upper=0.088655881867437475 effort=10.00 velocity=6.67 -> lower=0 upper=0.08865588186743747 effort=10.00 velocity=6.67; origin xyz=-0.03 -0.046499999999999986 0.026000000000000002 rpy=0 0 0 -> xyz=-0.075 -0.046499999999999986 0.026000000000000002 rpy=0 0 0
- joint black_key_42_joint: limit lower=0 upper=0.088655881867437475 effort=10.00 velocity=6.67 -> lower=0 upper=0.08865588186743747 effort=10.00 velocity=6.67; origin xyz=-0.03 -0.02299999999999991 0.026000000000000002 rpy=0 0 0 -> xyz=-0.075 -0.02299999999999991 0.026000000000000002 rpy=0 0 0
- joint black_key_45_joint: limit lower=0 upper=0.088655881867437475 effort=10.00 velocity=6.67 -> lower=0 upper=0.08865588186743747 effort=10.00 velocity=6.67; origin xyz=-0.03 0.02400000000000002 0.026000000000000002 rpy=0 0 0 -> xyz=-0.075 0.02400000000000002 0.026000000000000002 rpy=0 0 0
- joint black_key_47_joint: limit lower=0 upper=0.088655881867437475 effort=10.00 velocity=6.67 -> lower=0 upper=0.08865588186743747 effort=10.00 velocity=6.67; origin xyz=-0.03 0.0475000000000001 0.026000000000000002 rpy=0 0 0 -> xyz=-0.075 0.0475000000000001 0.026000000000000002 rpy=0 0 0
- joint black_key_49_joint: limit lower=0 upper=0.088655881867437475 effort=10.00 velocity=6.67 -> lower=0 upper=0.08865588186743747 effort=10.00 velocity=6.67; origin xyz=-0.03 0.07100000000000006 0.026000000000000002 rpy=0 0 0 -> xyz=-0.075 0.07100000000000006 0.026000000000000002 rpy=0 0 0
- joint black_key_4_joint: limit lower=0 upper=0.088655881867437475 effort=10.00 velocity=6.67 -> lower=0 upper=0.08865588186743747 effort=10.00 velocity=6.67; origin xyz=-0.03 -0.5399999999999999 0.026000000000000002 rpy=0 0 0 -> xyz=-0.075 -0.5399999999999999 0.026000000000000002 rpy=0 0 0
- joint black_key_52_joint: limit lower=0 upper=0.088655881867437475 effort=10.00 velocity=6.67 -> lower=0 upper=0.08865588186743747 effort=10.00 velocity=6.67; origin xyz=-0.03 0.118 0.026000000000000002 rpy=0 0 0 -> xyz=-0.075 0.118 0.026000000000000002 rpy=0 0 0
- joint black_key_54_joint: limit lower=0 upper=0.088655881867437475 effort=10.00 velocity=6.67 -> lower=0 upper=0.08865588186743747 effort=10.00 velocity=6.67; origin xyz=-0.03 0.14150000000000007 0.026000000000000002 rpy=0 0 0 -> xyz=-0.075 0.14150000000000007 0.026000000000000002 rpy=0 0 0
- joint black_key_57_joint: limit lower=0 upper=0.088655881867437475 effort=10.00 velocity=6.67 -> lower=0 upper=0.08865588186743747 effort=10.00 velocity=6.67; origin xyz=-0.03 0.1885 0.026000000000000002 rpy=0 0 0 -> xyz=-0.075 0.1885 0.026000000000000002 rpy=0 0 0
- joint black_key_59_joint: limit lower=0 upper=0.088655881867437475 effort=10.00 velocity=6.67 -> lower=0 upper=0.08865588186743747 effort=10.00 velocity=6.67; origin xyz=-0.03 0.21200000000000008 0.026000000000000002 rpy=0 0 0 -> xyz=-0.075 0.21200000000000008 0.026000000000000002 rpy=0 0 0
- joint black_key_61_joint: limit lower=0 upper=0.088655881867437475 effort=10.00 velocity=6.67 -> lower=0 upper=0.08865588186743747 effort=10.00 velocity=6.67; origin xyz=-0.03 0.23550000000000004 0.026000000000000002 rpy=0 0 0 -> xyz=-0.075 0.23550000000000004 0.026000000000000002 rpy=0 0 0
- joint black_key_64_joint: limit lower=0 upper=0.088655881867437475 effort=10.00 velocity=6.67 -> lower=0 upper=0.08865588186743747 effort=10.00 velocity=6.67; origin xyz=-0.03 0.2825000000000001 0.026000000000000002 rpy=0 0 0 -> xyz=-0.075 0.2825000000000001 0.026000000000000002 rpy=0 0 0
- joint black_key_66_joint: limit lower=0 upper=0.088655881867437475 effort=10.00 velocity=6.67 -> lower=0 upper=0.08865588186743747 effort=10.00 velocity=6.67; origin xyz=-0.03 0.30600000000000016 0.026000000000000002 rpy=0 0 0 -> xyz=-0.075 0.30600000000000016 0.026000000000000002 rpy=0 0 0
- joint black_key_69_joint: limit lower=0 upper=0.088655881867437475 effort=10.00 velocity=6.67 -> lower=0 upper=0.08865588186743747 effort=10.00 velocity=6.67; origin xyz=-0.03 0.353 0.026000000000000002 rpy=0 0 0 -> xyz=-0.075 0.353 0.026000000000000002 rpy=0 0 0
- joint black_key_6_joint: limit lower=0 upper=0.088655881867437475 effort=10.00 velocity=6.67 -> lower=0 upper=0.08865588186743747 effort=10.00 velocity=6.67; origin xyz=-0.03 -0.5164999999999998 0.026000000000000002 rpy=0 0 0 -> xyz=-0.075 -0.5164999999999998 0.026000000000000002 rpy=0 0 0
- joint black_key_71_joint: limit lower=0 upper=0.088655881867437475 effort=10.00 velocity=6.67 -> lower=0 upper=0.08865588186743747 effort=10.00 velocity=6.67; origin xyz=-0.03 0.37650000000000006 0.026000000000000002 rpy=0 0 0 -> xyz=-0.075 0.37650000000000006 0.026000000000000002 rpy=0 0 0
- joint black_key_73_joint: limit lower=0 upper=0.088655881867437475 effort=10.00 velocity=6.67 -> lower=0 upper=0.08865588186743747 effort=10.00 velocity=6.67; origin xyz=-0.03 0.4 0.026000000000000002 rpy=0 0 0 -> xyz=-0.075 0.4 0.026000000000000002 rpy=0 0 0
- joint black_key_76_joint: limit lower=0 upper=0.088655881867437475 effort=10.00 velocity=6.67 -> lower=0 upper=0.08865588186743747 effort=10.00 velocity=6.67; origin xyz=-0.03 0.44700000000000006 0.026000000000000002 rpy=0 0 0 -> xyz=-0.075 0.44700000000000006 0.026000000000000002 rpy=0 0 0
- joint black_key_78_joint: limit lower=0 upper=0.088655881867437475 effort=10.00 velocity=6.67 -> lower=0 upper=0.08865588186743747 effort=10.00 velocity=6.67; origin xyz=-0.03 0.47050000000000014 0.026000000000000002 rpy=0 0 0 -> xyz=-0.075 0.47050000000000014 0.026000000000000002 rpy=0 0 0
- joint black_key_81_joint: limit lower=0 upper=0.088655881867437475 effort=10.00 velocity=6.67 -> lower=0 upper=0.08865588186743747 effort=10.00 velocity=6.67; origin xyz=-0.03 0.5175000000000001 0.026000000000000002 rpy=0 0 0 -> xyz=-0.075 0.5175000000000001 0.026000000000000002 rpy=0 0 0
- joint black_key_83_joint: limit lower=0 upper=0.088655881867437475 effort=10.00 velocity=6.67 -> lower=0 upper=0.08865588186743747 effort=10.00 velocity=6.67; origin xyz=-0.03 0.5410000000000001 0.026000000000000002 rpy=0 0 0 -> xyz=-0.075 0.5410000000000001 0.026000000000000002 rpy=0 0 0
- joint black_key_85_joint: limit lower=0 upper=0.088655881867437475 effort=10.00 velocity=6.67 -> lower=0 upper=0.08865588186743747 effort=10.00 velocity=6.67; origin xyz=-0.03 0.5645000000000001 0.026000000000000002 rpy=0 0 0 -> xyz=-0.075 0.5645000000000001 0.026000000000000002 rpy=0 0 0
- joint black_key_9_joint: limit lower=0 upper=0.088655881867437475 effort=10.00 velocity=6.67 -> lower=0 upper=0.08865588186743747 effort=10.00 velocity=6.67; origin xyz=-0.03 -0.4695 0.026000000000000002 rpy=0 0 0 -> xyz=-0.075 -0.4695 0.026000000000000002 rpy=0 0 0
- joint white_key_0_joint: limit lower=0 upper=0.066568163775823808 effort=10.00 velocity=6.67 -> lower=0 upper=0.06656816377582381 effort=10.00 velocity=6.67; origin xyz=0.0 -0.59925 0.01125 rpy=0 0 0 -> xyz=-0.075 -0.59925 0.01125 rpy=0 0 0
- joint white_key_10_joint: limit lower=0 upper=0.066568163775823808 effort=10.00 velocity=6.67 -> lower=0 upper=0.06656816377582381 effort=10.00 velocity=6.67; origin xyz=0.0 -0.45824999999999994 0.01125 rpy=0 0 0 -> xyz=-0.075 -0.45824999999999994 0.01125 rpy=0 0 0
- joint white_key_12_joint: limit lower=0 upper=0.066568163775823808 effort=10.00 velocity=6.67 -> lower=0 upper=0.06656816377582381 effort=10.00 velocity=6.67; origin xyz=0.0 -0.43474999999999997 0.01125 rpy=0 0 0 -> xyz=-0.075 -0.43474999999999997 0.01125 rpy=0 0 0
- joint white_key_14_joint: limit lower=0 upper=0.066568163775823808 effort=10.00 velocity=6.67 -> lower=0 upper=0.06656816377582381 effort=10.00 velocity=6.67; origin xyz=0.0 -0.41124999999999995 0.01125 rpy=0 0 0 -> xyz=-0.075 -0.41124999999999995 0.01125 rpy=0 0 0
- joint white_key_15_joint: limit lower=0 upper=0.066568163775823808 effort=10.00 velocity=6.67 -> lower=0 upper=0.06656816377582381 effort=10.00 velocity=6.67; origin xyz=0.0 -0.38774999999999993 0.01125 rpy=0 0 0 -> xyz=-0.075 -0.38774999999999993 0.01125 rpy=0 0 0
- joint white_key_17_joint: limit lower=0 upper=0.066568163775823808 effort=10.00 velocity=6.67 -> lower=0 upper=0.06656816377582381 effort=10.00 velocity=6.67; origin xyz=0.0 -0.36424999999999996 0.01125 rpy=0 0 0 -> xyz=-0.075 -0.36424999999999996 0.01125 rpy=0 0 0
- joint white_key_19_joint: limit lower=0 upper=0.066568163775823808 effort=10.00 velocity=6.67 -> lower=0 upper=0.06656816377582381 effort=10.00 velocity=6.67; origin xyz=0.0 -0.34074999999999994 0.01125 rpy=0 0 0 -> xyz=-0.075 -0.34074999999999994 0.01125 rpy=0 0 0
- joint white_key_20_joint: limit lower=0 upper=0.066568163775823808 effort=10.00 velocity=6.67 -> lower=0 upper=0.06656816377582381 effort=10.00 velocity=6.67; origin xyz=0.0 -0.3172499999999999 0.01125 rpy=0 0 0 -> xyz=-0.075 -0.3172499999999999 0.01125 rpy=0 0 0
- joint white_key_22_joint: limit lower=0 upper=0.066568163775823808 effort=10.00 velocity=6.67 -> lower=0 upper=0.06656816377582381 effort=10.00 velocity=6.67; origin xyz=0.0 -0.29374999999999996 0.01125 rpy=0 0 0 -> xyz=-0.075 -0.29374999999999996 0.01125 rpy=0 0 0
- joint white_key_24_joint: limit lower=0 upper=0.066568163775823808 effort=10.00 velocity=6.67 -> lower=0 upper=0.06656816377582381 effort=10.00 velocity=6.67; origin xyz=0.0 -0.27024999999999993 0.01125 rpy=0 0 0 -> xyz=-0.075 -0.27024999999999993 0.01125 rpy=0 0 0
- joint white_key_26_joint: limit lower=0 upper=0.066568163775823808 effort=10.00 velocity=6.67 -> lower=0 upper=0.06656816377582381 effort=10.00 velocity=6.67; origin xyz=0.0 -0.24674999999999997 0.01125 rpy=0 0 0 -> xyz=-0.075 -0.24674999999999997 0.01125 rpy=0 0 0
- joint white_key_27_joint: limit lower=0 upper=0.066568163775823808 effort=10.00 velocity=6.67 -> lower=0 upper=0.06656816377582381 effort=10.00 velocity=6.67; origin xyz=0.0 -0.22324999999999995 0.01125 rpy=0 0 0 -> xyz=-0.075 -0.22324999999999995 0.01125 rpy=0 0 0
- joint white_key_29_joint: limit lower=0 upper=0.066568163775823808 effort=10.00 velocity=6.67 -> lower=0 upper=0.06656816377582381 effort=10.00 velocity=6.67; origin xyz=0.0 -0.19974999999999993 0.01125 rpy=0 0 0 -> xyz=-0.075 -0.19974999999999993 0.01125 rpy=0 0 0
- joint white_key_2_joint: limit lower=0 upper=0.066568163775823808 effort=10.00 velocity=6.67 -> lower=0 upper=0.06656816377582381 effort=10.00 velocity=6.67; origin xyz=0.0 -0.57575 0.01125 rpy=0 0 0 -> xyz=-0.075 -0.57575 0.01125 rpy=0 0 0
- joint white_key_31_joint: limit lower=0 upper=0.066568163775823808 effort=10.00 velocity=6.67 -> lower=0 upper=0.06656816377582381 effort=10.00 velocity=6.67; origin xyz=0.0 -0.17624999999999996 0.01125 rpy=0 0 0 -> xyz=-0.075 -0.17624999999999996 0.01125 rpy=0 0 0
- joint white_key_32_joint: limit lower=0 upper=0.066568163775823808 effort=10.00 velocity=6.67 -> lower=0 upper=0.06656816377582381 effort=10.00 velocity=6.67; origin xyz=0.0 -0.15274999999999994 0.01125 rpy=0 0 0 -> xyz=-0.075 -0.15274999999999994 0.01125 rpy=0 0 0
- joint white_key_34_joint: limit lower=0 upper=0.066568163775823808 effort=10.00 velocity=6.67 -> lower=0 upper=0.06656816377582381 effort=10.00 velocity=6.67; origin xyz=0.0 -0.12924999999999998 0.01125 rpy=0 0 0 -> xyz=-0.075 -0.12924999999999998 0.01125 rpy=0 0 0
- joint white_key_36_joint: limit lower=0 upper=0.066568163775823808 effort=10.00 velocity=6.67 -> lower=0 upper=0.06656816377582381 effort=10.00 velocity=6.67; origin xyz=0.0 -0.10574999999999996 0.01125 rpy=0 0 0 -> xyz=-0.075 -0.10574999999999996 0.01125 rpy=0 0 0
- joint white_key_38_joint: limit lower=0 upper=0.066568163775823808 effort=10.00 velocity=6.67 -> lower=0 upper=0.06656816377582381 effort=10.00 velocity=6.67; origin xyz=0.0 -0.08224999999999993 0.01125 rpy=0 0 0 -> xyz=-0.075 -0.08224999999999993 0.01125 rpy=0 0 0
- joint white_key_39_joint: limit lower=0 upper=0.066568163775823808 effort=10.00 velocity=6.67 -> lower=0 upper=0.06656816377582381 effort=10.00 velocity=6.67; origin xyz=0.0 -0.05874999999999997 0.01125 rpy=0 0 0 -> xyz=-0.075 -0.05874999999999997 0.01125 rpy=0 0 0
- joint white_key_3_joint: limit lower=0 upper=0.066568163775823808 effort=10.00 velocity=6.67 -> lower=0 upper=0.06656816377582381 effort=10.00 velocity=6.67; origin xyz=0.0 -0.5522499999999999 0.01125 rpy=0 0 0 -> xyz=-0.075 -0.5522499999999999 0.01125 rpy=0 0 0
- joint white_key_41_joint: limit lower=0 upper=0.066568163775823808 effort=10.00 velocity=6.67 -> lower=0 upper=0.06656816377582381 effort=10.00 velocity=6.67; origin xyz=0.0 -0.03524999999999989 0.01125 rpy=0 0 0 -> xyz=-0.075 -0.03524999999999989 0.01125 rpy=0 0 0
- joint white_key_43_joint: limit lower=0 upper=0.066568163775823808 effort=10.00 velocity=6.67 -> lower=0 upper=0.06656816377582381 effort=10.00 velocity=6.67; origin xyz=0.0 -0.011749999999999927 0.01125 rpy=0 0 0 -> xyz=-0.075 -0.011749999999999927 0.01125 rpy=0 0 0
- joint white_key_44_joint: limit lower=0 upper=0.066568163775823808 effort=10.00 velocity=6.67 -> lower=0 upper=0.06656816377582381 effort=10.00 velocity=6.67; origin xyz=0.0 0.011750000000000038 0.01125 rpy=0 0 0 -> xyz=-0.075 0.011750000000000038 0.01125 rpy=0 0 0
- joint white_key_46_joint: limit lower=0 upper=0.066568163775823808 effort=10.00 velocity=6.67 -> lower=0 upper=0.06656816377582381 effort=10.00 velocity=6.67; origin xyz=0.0 0.035250000000000004 0.01125 rpy=0 0 0 -> xyz=-0.075 0.035250000000000004 0.01125 rpy=0 0 0
- joint white_key_48_joint: limit lower=0 upper=0.066568163775823808 effort=10.00 velocity=6.67 -> lower=0 upper=0.06656816377582381 effort=10.00 velocity=6.67; origin xyz=0.0 0.05875000000000008 0.01125 rpy=0 0 0 -> xyz=-0.075 0.05875000000000008 0.01125 rpy=0 0 0
- joint white_key_50_joint: limit lower=0 upper=0.066568163775823808 effort=10.00 velocity=6.67 -> lower=0 upper=0.06656816377582381 effort=10.00 velocity=6.67; origin xyz=0.0 0.08225000000000005 0.01125 rpy=0 0 0 -> xyz=-0.075 0.08225000000000005 0.01125 rpy=0 0 0
- joint white_key_51_joint: limit lower=0 upper=0.066568163775823808 effort=10.00 velocity=6.67 -> lower=0 upper=0.06656816377582381 effort=10.00 velocity=6.67; origin xyz=0.0 0.10575000000000001 0.01125 rpy=0 0 0 -> xyz=-0.075 0.10575000000000001 0.01125 rpy=0 0 0
- joint white_key_53_joint: limit lower=0 upper=0.066568163775823808 effort=10.00 velocity=6.67 -> lower=0 upper=0.06656816377582381 effort=10.00 velocity=6.67; origin xyz=0.0 0.1292500000000001 0.01125 rpy=0 0 0 -> xyz=-0.075 0.1292500000000001 0.01125 rpy=0 0 0
- joint white_key_55_joint: limit lower=0 upper=0.066568163775823808 effort=10.00 velocity=6.67 -> lower=0 upper=0.06656816377582381 effort=10.00 velocity=6.67; origin xyz=0.0 0.15275000000000005 0.01125 rpy=0 0 0 -> xyz=-0.075 0.15275000000000005 0.01125 rpy=0 0 0
- joint white_key_56_joint: limit lower=0 upper=0.066568163775823808 effort=10.00 velocity=6.67 -> lower=0 upper=0.06656816377582381 effort=10.00 velocity=6.67; origin xyz=0.0 0.17625000000000002 0.01125 rpy=0 0 0 -> xyz=-0.075 0.17625000000000002 0.01125 rpy=0 0 0
- joint white_key_58_joint: limit lower=0 upper=0.066568163775823808 effort=10.00 velocity=6.67 -> lower=0 upper=0.06656816377582381 effort=10.00 velocity=6.67; origin xyz=0.0 0.1997500000000001 0.01125 rpy=0 0 0 -> xyz=-0.075 0.1997500000000001 0.01125 rpy=0 0 0
- joint white_key_5_joint: limit lower=0 upper=0.066568163775823808 effort=10.00 velocity=6.67 -> lower=0 upper=0.06656816377582381 effort=10.00 velocity=6.67; origin xyz=0.0 -0.5287499999999999 0.01125 rpy=0 0 0 -> xyz=-0.075 -0.5287499999999999 0.01125 rpy=0 0 0
- joint white_key_60_joint: limit lower=0 upper=0.066568163775823808 effort=10.00 velocity=6.67 -> lower=0 upper=0.06656816377582381 effort=10.00 velocity=6.67; origin xyz=0.0 0.22325000000000006 0.01125 rpy=0 0 0 -> xyz=-0.075 0.22325000000000006 0.01125 rpy=0 0 0
- joint white_key_62_joint: limit lower=0 upper=0.066568163775823808 effort=10.00 velocity=6.67 -> lower=0 upper=0.06656816377582381 effort=10.00 velocity=6.67; origin xyz=0.0 0.24675000000000002 0.01125 rpy=0 0 0 -> xyz=-0.075 0.24675000000000002 0.01125 rpy=0 0 0
- joint white_key_63_joint: limit lower=0 upper=0.066568163775823808 effort=10.00 velocity=6.67 -> lower=0 upper=0.06656816377582381 effort=10.00 velocity=6.67; origin xyz=0.0 0.2702500000000001 0.01125 rpy=0 0 0 -> xyz=-0.075 0.2702500000000001 0.01125 rpy=0 0 0
- joint white_key_65_joint: limit lower=0 upper=0.066568163775823808 effort=10.00 velocity=6.67 -> lower=0 upper=0.06656816377582381 effort=10.00 velocity=6.67; origin xyz=0.0 0.29375000000000007 0.01125 rpy=0 0 0 -> xyz=-0.075 0.29375000000000007 0.01125 rpy=0 0 0
- joint white_key_67_joint: limit lower=0 upper=0.066568163775823808 effort=10.00 velocity=6.67 -> lower=0 upper=0.06656816377582381 effort=10.00 velocity=6.67; origin xyz=0.0 0.31725000000000003 0.01125 rpy=0 0 0 -> xyz=-0.075 0.31725000000000003 0.01125 rpy=0 0 0
- joint white_key_68_joint: limit lower=0 upper=0.066568163775823808 effort=10.00 velocity=6.67 -> lower=0 upper=0.06656816377582381 effort=10.00 velocity=6.67; origin xyz=0.0 0.34075 0.01125 rpy=0 0 0 -> xyz=-0.075 0.34075 0.01125 rpy=0 0 0
- joint white_key_70_joint: limit lower=0 upper=0.066568163775823808 effort=10.00 velocity=6.67 -> lower=0 upper=0.06656816377582381 effort=10.00 velocity=6.67; origin xyz=0.0 0.3642500000000001 0.01125 rpy=0 0 0 -> xyz=-0.075 0.3642500000000001 0.01125 rpy=0 0 0
- joint white_key_72_joint: limit lower=0 upper=0.066568163775823808 effort=10.00 velocity=6.67 -> lower=0 upper=0.06656816377582381 effort=10.00 velocity=6.67; origin xyz=0.0 0.38775000000000004 0.01125 rpy=0 0 0 -> xyz=-0.075 0.38775000000000004 0.01125 rpy=0 0 0
- joint white_key_74_joint: limit lower=0 upper=0.066568163775823808 effort=10.00 velocity=6.67 -> lower=0 upper=0.06656816377582381 effort=10.00 velocity=6.67; origin xyz=0.0 0.41125 0.01125 rpy=0 0 0 -> xyz=-0.075 0.41125 0.01125 rpy=0 0 0
- joint white_key_75_joint: limit lower=0 upper=0.066568163775823808 effort=10.00 velocity=6.67 -> lower=0 upper=0.06656816377582381 effort=10.00 velocity=6.67; origin xyz=0.0 0.4347500000000001 0.01125 rpy=0 0 0 -> xyz=-0.075 0.4347500000000001 0.01125 rpy=0 0 0
- joint white_key_77_joint: limit lower=0 upper=0.066568163775823808 effort=10.00 velocity=6.67 -> lower=0 upper=0.06656816377582381 effort=10.00 velocity=6.67; origin xyz=0.0 0.45825000000000016 0.01125 rpy=0 0 0 -> xyz=-0.075 0.45825000000000016 0.01125 rpy=0 0 0
- joint white_key_79_joint: limit lower=0 upper=0.066568163775823808 effort=10.00 velocity=6.67 -> lower=0 upper=0.06656816377582381 effort=10.00 velocity=6.67; origin xyz=0.0 0.48175 0.01125 rpy=0 0 0 -> xyz=-0.075 0.48175 0.01125 rpy=0 0 0
- joint white_key_7_joint: limit lower=0 upper=0.066568163775823808 effort=10.00 velocity=6.67 -> lower=0 upper=0.06656816377582381 effort=10.00 velocity=6.67; origin xyz=0.0 -0.50525 0.01125 rpy=0 0 0 -> xyz=-0.075 -0.50525 0.01125 rpy=0 0 0
- joint white_key_80_joint: limit lower=0 upper=0.066568163775823808 effort=10.00 velocity=6.67 -> lower=0 upper=0.06656816377582381 effort=10.00 velocity=6.67; origin xyz=0.0 0.5052500000000001 0.01125 rpy=0 0 0 -> xyz=-0.075 0.5052500000000001 0.01125 rpy=0 0 0
- joint white_key_82_joint: limit lower=0 upper=0.066568163775823808 effort=10.00 velocity=6.67 -> lower=0 upper=0.06656816377582381 effort=10.00 velocity=6.67; origin xyz=0.0 0.5287500000000002 0.01125 rpy=0 0 0 -> xyz=-0.075 0.5287500000000002 0.01125 rpy=0 0 0
- joint white_key_84_joint: limit lower=0 upper=0.066568163775823808 effort=10.00 velocity=6.67 -> lower=0 upper=0.06656816377582381 effort=10.00 velocity=6.67; origin xyz=0.0 0.55225 0.01125 rpy=0 0 0 -> xyz=-0.075 0.55225 0.01125 rpy=0 0 0
- joint white_key_86_joint: limit lower=0 upper=0.066568163775823808 effort=10.00 velocity=6.67 -> lower=0 upper=0.06656816377582381 effort=10.00 velocity=6.67; origin xyz=0.0 0.5757500000000001 0.01125 rpy=0 0 0 -> xyz=-0.075 0.5757500000000001 0.01125 rpy=0 0 0
- joint white_key_87_joint: limit lower=0 upper=0.066568163775823808 effort=10.00 velocity=6.67 -> lower=0 upper=0.06656816377582381 effort=10.00 velocity=6.67; origin xyz=0.0 0.59925 0.01125 rpy=0 0 0 -> xyz=-0.075 0.59925 0.01125 rpy=0 0 0
- joint white_key_8_joint: limit lower=0 upper=0.066568163775823808 effort=10.00 velocity=6.67 -> lower=0 upper=0.06656816377582381 effort=10.00 velocity=6.67; origin xyz=0.0 -0.48174999999999996 0.01125 rpy=0 0 0 -> xyz=-0.075 -0.48174999999999996 0.01125 rpy=0 0 0
